Commit message: wip: 改完第一版暂存，没测

File: src/srm27_navigation/srm27_nav_bringup/urdf/sentry_robot_cylinder.xacro (robot description, xacro)
@@ -7,9 +7,11 @@
     不要再回头改 srm_auto_sentry 那一份。
   注意:
-    下面 livox_frame 的 mesh 写的是 package://pb_rm_simulation/meshes/mid360.stl，
-    而 pb_rm_simulation 不在本工作空间。real_mapping_launch.py 与
-    real_robot_state_publisher_launch.py 加载时会把它改写为本包的
-    package://srm27_nav_bringup/meshes/mid360.stl（副本见 ../meshes/mid360.stl）。
-    若把本文件直接交给别的工具使用，需自行处理这个 URI。
+    本文件是实车链路使用的 URDF 入口；仿真使用的 SDF 由
+    srm27_robot_description 依据 config/srm27_sentry_geometry.yaml 生成，
+    几何数值必须保持一致。
+    livox_frame 的 mesh 指向 srm27_robot_description 包内的 mid360.stl 副本，
+    不再引用不在本工作空间的 package://pb_rm_simulation/。
+    real_mapping_launch.py 与 real_robot_state_publisher_launch.py 加载时
+    仍会把历史遗留的 package://pb_rm_simulation/ 前缀改写为描述包内的路径。
 -->
 <robot name="robot"
@@ -152,5 +154,5 @@
       <origin xyz="0.025 -0.0265 -0.025" rpy="${pi/2} 0 ${pi}"/>
       <geometry>
-        <mesh filename="package://pb_rm_simulation/meshes/mid360.stl" scale="0.001 0.001 0.001"/>
+        <mesh filename="package://srm27_robot_description/meshes/mid360.stl" scale="0.001 0.001 0.001"/>
       </geometry>
       <material name="blue">
